File: 11_Joystick.kicad_pcb (KiCad board)
At the start: 2 copper layers, 65 x 25 mm, 11 parts, among them J1 Conn_01x04, U1 MCP3426-xSN, U2 joystick

Commit message: maj split librairie
Parts:
- U2: footprint Chimere:RKJXV1220 -> Chimere_comps:RKJXV1220
